Commit message: Simplified meshes

File: skratch_description/description/base/skratch_base.xacro (robot description, xacro)
@@ -1,15 +1,15 @@
 <?xml version="1.0"?>
-<robot name="skratch_wheel_support" xmlns:xacro="http://www.ros.org/wiki/xacro">
-    <xacro:macro name="skratch_wheel_support" params="name">
+<robot name="skratch_base" xmlns:xacro="http://www.ros.org/wiki/xacro">
+    <xacro:macro name="skratch_base" params="name">
         <link name="${name}">
             <inertial>
-                <origin xyz="-0.1 0.0 -0.008" rpy="0.0 -0.0 0.0" />
-                <mass value="1.0" />
-                <inertia ixx="0.0213197" iyy="0.0224124" izz="0.0012279" ixy="0.0" iyz="0.0" ixz="0.0" />
+                <mass value="2.0"/>
+                <origin xyz="0 0 0" rpy="0 0 0"/>
+                <inertia ixx="0.03287973" iyy="0.06900190" izz="0.09325417" ixy="0.0" ixz="0.0" iyz="0.0"/>
             </inertial>
             <visual>
                 <origin xyz="0.0 0.0 0.0" rpy="0.0 0.0 0.0" />
                 <geometry>
-                    <mesh filename="file://$(find skratch_description)/meshes/base/skratch_wheel_support.stl" scale="0.001 0.001 0.001"/>
+                    <mesh filename="file://$(find skratch_description)/meshes/base/skratch_base.stl" scale="0.001 0.001 0.001"/>
                 </geometry>
                 <material name="Grey">
@@ -20,5 +20,5 @@
                 <origin xyz="0.0 0.0 0.0" rpy="0.0 0.0 0.0" />
                 <geometry>
-                    <mesh filename="file://$(find skratch_description)/meshes/base/skratch_wheel_support.stl" scale="0.001 0.001 0.001"/>
+                    <mesh filename="file://$(find skratch_description)/meshes/base/skratch_base.stl" scale="0.001 0.001 0.001"/>
                 </geometry>
             </collision>

File: skratch_description/description/skratch_robot.urdf.xacro (robot description, xacro)
@@ -1,96 +1,64 @@
 <?xml version="1.0" ?>
 <robot name="skratch_base" xmlns:xacro="http://www.ros.org/wiki/xacro">
-    <xacro:include filename="base/skratch_bottom_base.xacro"/>
-    <xacro:include filename="base/skratch_top_base.xacro"/>
-    <xacro:include filename="base/skratch_wheel_support.xacro"/>
+    <xacro:include filename="base/skratch_base.xacro"/>
     <xacro:include filename="wheels/kelo_drive_top_part.xacro"/>
     <xacro:include filename="lidar/lidar.xacro"/>
-    <xacro:include filename="$(find skratch_gazebo)/gazebo/skratch_gazebo.xacro"/>
+    <!-- <xacro:include filename="$(find skratch_gazebo)/gazebo/skratch_gazebo.xacro"/> -->
     <xacro:include filename="base/skratch_base_plate.xacro"/>
-    <xacro:include filename="$(find kinova_arm_description)/description/kinova_arm_macro.xacro"/>
-    <xacro:include filename="$(find kinova_arm_gazebo)/gazebo/kinova_arm_ros2_control.xacro"/>
-    <xacro:kinova_arm_ros2_control name="kinova_arm" initial_positions_file="$(find kinova_arm_gazebo)/config/initial_positions.yaml"/>
+    <!-- <xacro:include filename="$(find kinova_arm_description)/description/kinova_arm_macro.xacro"/> -->
+    <!-- <xacro:include filename="$(find kinova_arm_gazebo)/gazebo/kinova_arm_ros2_control.xacro"/> -->
+    <!-- <xacro:kinova_arm_ros2_control name="kinova_arm" initial_positions_file="$(find kinova_arm_gazebo)/config/initial_positions.yaml"/> -->
     <link name="base_link"></link>
-    <xacro:skratch_top_base name="skratch_left_top_base"/>
-    <joint name="base_joint" type="fixed">
-        <origin xyz="0.0 -0.005 0.15" rpy="0.0 0.0 0.0"/>
+    <xacro:skratch_base name="skratch_base"/>
+    <joint name="base_link_joint" type="fixed">
+        <origin xyz="0.0 0.0 0.0" rpy="0.0 0.0 0.0"/>
         <parent link="base_link"/>
-        <child link="skratch_left_top_base"/>
-    </joint>
-    <xacro:skratch_top_base name="skratch_right_top_base"/>
-    <joint name="right_top_base_joint" type="fixed">
-        <origin xyz="0.0 0.003 0.15" rpy="0.0 0.0 3.14"/>
-        <parent link="base_link"/>
-        <child link="skratch_right_top_base"/>
-    </joint>
-    <xacro:skratch_bottom_base name="skratch_left_bottom_base"/>
-    <joint name="left_bottom_base_joint" type="fixed">
-        <origin xyz="0.0 -0.099 -0.138" rpy="3.14 0.0 0.0"/>
-        <parent link="skratch_left_top_base"/>
-        <child link="skratch_left_bottom_base"/>
-    </joint>
-    <xacro:skratch_bottom_base name="skratch_right_bottom_base"/>
-    <joint name="right_bottom_base_joint" type="fixed">
-        <origin xyz="0.0 -0.099 -0.138" rpy="3.14 0.0 0.0"/>
-        <parent link="skratch_right_top_base"/>
-        <child link="skratch_right_bottom_base"/>
-    </joint>
-    <xacro:skratch_wheel_support name="skratch_left_wheel_support"/>
-    <joint name="left_wheel_support_joint" type="fixed">
-        <origin xyz="0.0 0.0 -0.1022" rpy="0.0 0.0 0.0"/>
-        <parent link="skratch_left_bottom_base"/>
-        <child link="skratch_left_wheel_support"/>
-    </joint>
-    <xacro:skratch_wheel_support name="skratch_right_wheel_support"/>
-    <joint name="right_wheel_support_joint" type="fixed">
-        <origin xyz="0.0 0.0 -0.1022" rpy="0.0 0.0 0.0"/>
-        <parent link="skratch_right_bottom_base"/>
-        <child link="skratch_right_wheel_support"/>
+        <child link="skratch_base"/>
     </joint>
     <xacro:skratch_base_plate name="skratch_arm_base_plate"/>
     <joint name="arm_base_plate_joint" type="fixed">
-        <origin xyz="0.2115 0.005 0.023" rpy="0.0 0.0 0.0"/>
-        <parent link="skratch_left_top_base"/>
+        <origin xyz="0.2115 0.005 0.16" rpy="0.0 0.0 0.0"/>
+        <parent link="skratch_base"/>
         <child link="skratch_arm_base_plate"/>
     </joint>
-    <xacro:kinova_arm/>
+    <!-- <xacro:kinova_arm/>
     <joint name="kinova_arm_base_joint" type="fixed">
         <origin xyz="0.0 0.0 0.0" rpy="1.57 0 3.14"/>
         <parent link="skratch_arm_base_plate"/>
         <child link="kinova_base"/>
-    </joint>
-    <xacro:kelo_drive_top_part name="front_left_drive_top_part" parent="skratch_left_wheel_support" drive_name="skratch_1_drive">
-        <origin xyz="0.202 0 0.018" rpy="3.14 0 0.0"/>
+    </joint> -->
+    <xacro:kelo_drive_top_part name="front_left_drive_top_part" parent="skratch_base" drive_name="skratch_1_drive">
+        <origin xyz="0.202 0.118 0.0" rpy="0.0 0 0.0"/>
     </xacro:kelo_drive_top_part>
-    <xacro:kelo_drive_top_part name="front_right_drive_top_part" parent="skratch_right_wheel_support" drive_name="skratch_2_drive">
-        <origin xyz="-0.202 0 0.018" rpy="3.14 0 0.0"/>
+    <xacro:kelo_drive_top_part name="front_right_drive_top_part" parent="skratch_base" drive_name="skratch_2_drive">
+        <origin xyz="0.202 -0.118 0.0" rpy="0.0 0 0.0"/>
     </xacro:kelo_drive_top_part>
-    <xacro:kelo_drive_top_part name="rear_left_drive_top_part" parent="skratch_left_wheel_support" drive_name="skratch_3_drive">
-        <origin xyz="-0.202 0 0.018" rpy="3.14 0 0.0"/>
+    <xacro:kelo_drive_top_part name="rear_left_drive_top_part" parent="skratch_base" drive_name="skratch_3_drive">
+        <origin xyz="-0.202 0.118 0.0" rpy="0.0 0 0.0"/>
     </xacro:kelo_drive_top_part>
-    <xacro:kelo_drive_top_part name="rear_right_drive_top_part" parent="skratch_right_wheel_support" drive_name="skratch_4_drive">
-        <origin xyz="0.202 0 0.018" rpy="3.14 0 0.0"/>
+    <xacro:kelo_drive_top_part name="rear_right_drive_top_part" parent="skratch_base" drive_name="skratch_4_drive">
+        <origin xyz="-0.202 -0.118 0.0" rpy="0.0 0 0.0"/>
     </xacro:kelo_drive_top_part>
-    <xacro:lidar name="front_lidar"/>
+    <!-- <xacro:lidar name="front_lidar"/>
     <joint name="front_lidar_joint" type="fixed">
         <origin xyz="0.318 -0.203 -0.1635" rpy="0.0 0.0 0.820305"/>
-        <parent link="skratch_left_top_base"/>
+        <parent link="skratch_base"/>
         <child link="front_lidar"/>
         <axis xyz="0.0 0.0 1.0"/>
-    </joint>
-    <xacro:lidar name="rear_lidar"/>
+    </joint> -->
+    <!-- <xacro:lidar name="rear_lidar"/>
     <joint name="rear_lidar_joint" type="fixed">
         <origin xyz="0.318 -0.203 -0.1635" rpy="0.0 0.0 2.3214"/>
-        <parent link="skratch_right_top_base"/>
+        <parent link="skratch_base"/>
         <child link="rear_lidar"/>
         <axis xyz="0.0 0.0 1.0"/>
-    </joint>
+    </joint> -->
     <xacro:skratch_base_plate name="skratch_battery_base_plate"/>
     <joint name="battery_base_plate_joint" type="fixed">
         <origin xyz="-0.2115 0.005 0.023" rpy="0.0 0.0 3.1416"/>
-        <parent link="skratch_left_top_base"/>
+        <parent link="skratch_base"/>
         <child link="skratch_battery_base_plate"/>
     </joint>
-    <link name="battery_link">
+    <!-- <link name="battery_link">
         <visual>
             <geometry>
@@ -120,4 +88,4 @@
         <child link="battery_link"/>
         <axis xyz="0.0 0.0 1.0"/>
-    </joint>
+    </joint> -->
 </robot>

File: skratch_description/description/wheels/kelo_drive.xacro (robot description, xacro)
@@ -25,5 +25,5 @@
             </inertial>
         </link>
-        <joint name="${name}_pivot_joint" type="fixed">
+        <joint name="${name}_pivot_joint" type="continuous">
             <xacro:insert_block name="origin" />
             <axis xyz="0 0 1"/>

File: skratch_description/description/wheels/kelo_drive_top_part.xacro (robot description, xacro)
@@ -5,5 +5,5 @@
         <link name="${name}_drive_top_part">
             <visual>
-                <origin xyz="0 0 0" rpy="0 0 0"/>
+                <origin xyz="0 0 0.081" rpy="0 0 0"/>
                 <geometry>
                     <mesh filename="file://$(find skratch_description)/meshes/wheels/kelo_drive_top_part.dae" scale="1 1 1"/>
@@ -14,5 +14,5 @@
             </visual>
             <collision>
-                <origin xyz="0 0 0" rpy="0 0 0"/>
+                <origin xyz="0 0 0.081" rpy="0 0 0"/>
                 <geometry>
                     <mesh filename="file://$(find skratch_description)/meshes/wheels/kelo_drive_top_part.dae" scale="1 1 1"/>
@@ -31,5 +31,5 @@
         </joint>
         <xacro:kelo_drive name="${drive_name}" parent="${name}_drive_top_part">
-            <origin xyz="0 0 -0.09" rpy="0 0 0.0"/>
+            <origin xyz="0 0 -0.01" rpy="0 0 0.0"/>
         </xacro:kelo_drive>
     </xacro:macro>

File: skratch_gazebo/gazebo/skratch_gazebo.xacro (robot description, xacro)
@@ -55,5 +55,5 @@
                         <resolution>1</resolution>
                         <min_angle>5.2</min_angle>
-		                <max_angle>1.2</max_angle>
+                        <max_angle>1.2</max_angle>
                     </horizontal>
                 </scan>
